Commit message: UR_Compliance

File: diff_drive_controller/test/sphere_wheel.xacro (robot description, xacro)
@@ -1,5 +1,5 @@
 <?xml version="1.0"?>
 <robot xmlns:xacro="http://www.ros.org/wiki/xacro">
-  <macro name="sphere_wheel" params="name parent radius *origin">
+  <xacro:macro name="sphere_wheel" params="name parent radius *origin">
     <link name="${name}_link">
       <inertial>
@@ -24,5 +24,5 @@
       <parent link="${parent}_link"/>
       <child link="${name}_link"/>
-      <insert_block name="origin"/>
+      <xacro:insert_block name="origin"/>
       <axis xyz="0 0 1"/>
     </joint>
@@ -37,4 +37,4 @@
       <material>Gazebo/Red</material>
     </gazebo>
-  </macro>
+  </xacro:macro>
 </robot>

File: diff_drive_controller/test/wheel.xacro (robot description, xacro)
@@ -1,5 +1,5 @@
 <?xml version="1.0"?>
 <robot xmlns:xacro="http://www.ros.org/wiki/xacro">
-  <macro name="wheel" params="name parent radius thickness *origin">
+  <xacro:macro name="wheel" params="name parent radius thickness *origin">
     <link name="${name}_link">
       <inertial>
@@ -24,5 +24,5 @@
       <parent link="${parent}_link"/>
       <child link="${name}_link"/>
-      <insert_block name="origin"/>
+      <xacro:insert_block name="origin"/>
       <axis xyz="0 0 1"/>
     </joint>
@@ -37,4 +37,4 @@
       <material>Gazebo/Red</material>
     </gazebo>
-  </macro>
+  </xacro:macro>
 </robot>
